Commit message: code cleaning

File: urdf/waiter.urdf.xacro (robot description, xacro)
@@ -37,14 +37,4 @@
       <child link="legs_link"/>
     </joint>
-    <!-- <transmission name="trans_base_to_legs">
-      <type>transmission_interface/SimpleTransmission</type>
-      <joint name="base_to_legs">
-        <hardwareInterface>EffortJointInterface</hardwareInterface>
-      </joint>
-      <actuator name="motor_base_to_legs">
-        <mechanicalReduction>0.5</mechanicalReduction>
-        <hardwareInterface>EffortJointInterface</hardwareInterface>
-      </actuator>
-    </transmission> -->
     <link name="legs_link">
       <visual>
@@ -68,14 +58,4 @@
       <child link="body_link"/>
     </joint>
-    <!-- <transmission name="trans_legs_to_body">
-      <type>transmission_interface/SimpleTransmission</type>
-      <joint name="legs_to_body">
-        <hardwareInterface>EffortJointInterface</hardwareInterface>
-      </joint>
-      <actuator name="motor_legs_to_body">
-        <mechanicalReduction>0.5</mechanicalReduction>
-        <hardwareInterface>EffortJointInterface</hardwareInterface>
-      </actuator>
-    </transmission> -->
     <link name="body_link">
       <visual>
@@ -94,7 +74,3 @@
       <xacro:default_inertial mass="10"/>
     </link>
-    <!-- <gazebo>
-      <plugin name="gazebo_ros_control" filename="libgazebo_ros_control.so">
-      </plugin>
-    </gazebo> -->
 </robot>

Commit message: urdf updated

File: urdf/waiter.urdf.xacro (robot description, xacro)
@@ -2,7 +2,8 @@
 <robot name="waiterobot" xmlns:xacro="http://ros.org/wiki/xacro">
     <xacro:property name="width" value="0.2" />
-    <xacro:property name="baselen" value="0.2" />
-    <xacro:property name="bodylen" value="0.6" />
-    <xacro:property name="legslen" value="1.0" />
+    <xacro:property name="base_thickness" value="0.2" />
+    <xacro:property name="base_len" value="0.5" />
+    <xacro:property name="body_height" value="0.6" />
+    <xacro:property name="legs_height" value="1.0" />
     <xacro:property name="pi" value="3.14159265" />
     <material name="red">
@@ -25,6 +26,5 @@
         <origin rpy="0.0 0.0 0.0" xyz="0.0 0.0 0.0"/>
         <geometry>
-          <!-- <cylinder length="${baselen}" radius="${width}"/> -->
-          <box size="0.5 0.5 ${baselen}"/>
+          <box size="${base_len} ${base_len} ${base_thickness}"/>
         </geometry>
         <material name="white"/>
@@ -39,7 +39,8 @@
     <link name="legs_link">
       <visual>
-        <origin rpy="0.0 0.0 0.0" xyz="0.0 0.0 ${baselen+0.2}"/>
+        <origin rpy="0.0 0.0 0.0" xyz="0.0 0.0 ${base_thickness+0.2}"/>
         <geometry>
-          <cylinder radius="${width}" length="${legslen}"/>
+          <!-- <cylinder radius="${width}" length="${legs_height}"/> -->
+          <box size="${width} ${width*2.4} ${legs_height}"/>
         </geometry>
         <material name="black"/>
@@ -47,5 +48,6 @@
       <collision>
         <geometry>
-          <cylinder radius="${width}" length="${legslen}"/>
+          <!-- <cylinder radius="${width}" length="${legs_height}"/> -->
+          <box size="${width} ${width*2.4} ${legs_height}"/>
         </geometry>
       </collision>
@@ -54,5 +56,5 @@
     <joint name="legs_to_body" type="revolute">
       <axis xyz="1 0 0"/>
-      <limit lower="0.0" upper="${pi/4.0}" effort="50.0" velocity="0.5"/>
+      <limit lower="0.0" upper="${pi/16.0}" effort="50.0" velocity="0.5"/>
       <parent link="legs_link"/>
       <child link="body_link"/>
@@ -60,8 +62,8 @@
     <link name="body_link">
       <visual>
-        <origin xyz="0.0 0.0 ${legslen+0.1}" rpy="0.0 0.0 0.0"/>
+        <origin xyz="0.2 0.0 ${legs_height}" rpy="0.0 0.0 0.0"/>
         <geometry>
-          <!-- <cylinder radius="${width}" length="${bodylen}"/> -->
-          <box size="${width} ${width} ${bodylen}"/>
+          <!-- <cylinder radius="${width}" length="${body_height}"/> -->
+          <box size="${width} ${width} ${body_height}"/>
         </geometry>
         <material name="red"/>
@@ -69,5 +71,5 @@
       <collision>
         <geometry>
-          <cylinder radius="${width}" length="${bodylen}"/>
+          <box size="${width} ${width} ${body_height}"/>
         </geometry>
       </collision>

Commit message: Head and hair links added,  rate frequency of moving joints changed from 10hz to 1hz

File: urdf/waiter.urdf.xacro (robot description, xacro)
@@ -2,4 +2,7 @@
 <robot name="waiterobot" xmlns:xacro="http://ros.org/wiki/xacro">
     <xacro:property name="width" value="0.2" />
+    <xacro:property name="head_radius" value="0.25" />
+    <xacro:property name="head_len" value="0.4" />
+    <xacro:property name="hair_len" value="0.07" />
     <xacro:property name="base_thickness" value="0.2" />
     <xacro:property name="base_len" value="0.5" />
@@ -9,4 +12,7 @@
     <material name="red">
         <color rgba="1 0 0 1"/>
+    </material>
+    <material name="skin_color">
+        <color rgba="0.925 0.737 0.706 1"/>
     </material>
     <material name="black">
@@ -76,3 +82,43 @@
       <xacro:default_inertial mass="10"/>
     </link>
+    <joint name="body_to_head" type="fixed">
+      <parent link="body_link"/>
+      <child link="head_link"/>
+      <origin xyz="0 0 0"/>
+    </joint>
+    <link name="head_link">
+      <visual>
+        <origin xyz="0.2 0.0 ${legs_height+body_height-0.2}" rpy="0.0 0.0 0.0"/>
+        <geometry>
+          <cylinder length="${head_len}" radius="${head_radius}"/>
+        </geometry>
+        <material name="skin_color"/>
+      </visual>
+      <collision>
+        <geometry>
+          <cylinder length="${head_len}" radius="${head_radius}"/>
+        </geometry>
+      </collision>
+      <xacro:default_inertial mass="4"/>
+    </link>
+    <joint name="head_to_hair" type="fixed">
+      <parent link="head_link"/>
+      <child link="hair_link"/>
+      <origin xyz="0 0 0"/>
+    </joint>
+    <link name="hair_link">
+      <visual>
+        <origin xyz="0.2 0.0 ${legs_height+body_height+0.05}" rpy="0.0 0.0 0.0"/>
+        <geometry>
+          <cylinder length="${hair_len}" radius="${head_radius}"/>
+        </geometry>
+        <material name="black"/>
+      </visual>
+      <collision>
+        <geometry>
+          <box size="${width} ${width} ${body_height}"/>
+        </geometry>
+      </collision>
+      <xacro:default_inertial mass="4"/>
+    </link>
 </robot>
